File: Hardware/OpenThermMonitorTwomes.sch (KiCad schematic (older format))
At the start: 28 parts, among them J1 Boiler, J2 Therm, P1 CONN_01X08, P2 CONN_01X08, SW1 SW_Push, U1 HT7550-1, U2 LM393DR2G, U3 EL357N(C), U4 EL357N(C)

Commit message: V1.1 Fixed risetime issue
Parts:
- C1: value 100nF -> 10nF; symbol jlcpcb-basic-mlcc-0603:100nF -> jlcpcb-basic-mlcc-0603:10nF; C57112 (none) -> C57112; LCSC C14663 -> (none)
- R8: value 470R -> 1k; symbol jlcpcb-basic-resistor-0603:470R -> jlcpcb-basic-resistor-0603:1k; LCSC C23179 -> C21190
Other:
- note added: "2021-08-26 V1.1"
- note added: "20210826 V1.1:\nChanges: \nC1 from 100 nF to 10 nF to reduce rise time of VDC\nR8 from 470R to 1k to reduce current consumption blue voltage/therm/master LED (sufficient for EL357NC)\nFootprints same, still compatible with PCB 20210708 V1.0"
- note added: "Author:\nMarco Winkelman\nWindesheim University of Applied Science\nLectoraat Energietransitie\n\nLicensed under CERN-OHL-P v2"
- note removed: "2021-04-28"
- note removed: "Author:\nMarco Winkelman\nWindesheim University of Applied Science\nLectoraat Energietransitie"
- note removed: "Rev 0.2"
Changed lines of the file:
@@
 Connection ~ 2700 4000
 Connection ~ 3050 4000
-Text Notes 7050 6950 0    50   ~ 0
-Author:\nMarco Winkelman\nWindesheim University of Applied Science\nLectoraat Energietransitie
-Text Notes 8150 7650 0    50   ~ 0
-2021-04-28
+Text Notes 7050 7050 0    50   ~ 0
+Author:\nMarco Winkelman\nWindesheim University of Applied Science\nLectoraat Energietransitie\n\nLicensed under CERN-OHL-P v2
 Text Label 5900 4800 0    50   ~ 0
 MasterCommands
@@
 $EndComp
 $Comp
-L jlcpcb-basic-mlcc-0603:100nF C1
+L jlcpcb-basic-mlcc-0603:10nF C1
 U 1 1 6087E72A
 P 2350 3550
 F 0 "C1" H 2442 3596 50  0000 L CNN
-F 1 "100nF" H 2442 3505 50  0000 L CNN
+F 1 "10nF" H 2442 3505 50  0000 L CNN
 F 2 "Capacitor_SMD:C_0603_1608Metric" H 2388 3400 50  0001 C CNN
 F 3 "https://datasheet.lcsc.com/szlcsc/YAGEO-CC0603KRX7R9BB104_C14663.pdf" V 2350 3550 50  0001 C CNN
-F 4 "C14663" V 2350 3550 50  0001 C CNN "LCSC"
+F 4 "C57112" V 2350 3550 50  0001 C CNN "C57112"
 	1    2350 3550
 	1    0    0    -1
@@
 $EndComp
 $Comp
-L jlcpcb-basic-resistor-0603:470R R8
+L jlcpcb-basic-resistor-0603:1k R8
 U 1 1 6090D18C
 P 4400 4800
 F 0 "R8" H 4341 4754 50  0000 R CNN
-F 1 "470R" H 4341 4845 50  0000 R CNN
+F 1 "1k" H 4341 4845 50  0000 R CNN
 F 2 "Resistor_SMD:R_0603_1608Metric" V 4330 4800 50  0001 C CNN
 F 3 "https://datasheet.lcsc.com/szlcsc/Uniroyal-Elec-0603WAF4700T5E_C23179.pdf" V 4400 4800 50  0001 C CNN
-F 4 "C23179" V 4400 4800 50  0001 C CNN "LCSC"
+F 4 "C21190" V 4400 4800 50  0001 C CNN "LCSC"
 	1    4400 4800
 	0    -1   -1   0
@@
 Wire Wire Line
 	4500 3600 4500 4600
-Text Notes 8600 7500 0    50   ~ 0
-Rev 0.2
+Text Notes 5250 3000 0    50   ~ 0
+20210826 V1.1:\nChanges:  \nC1 from 100 nF to 10 nF to reduce rise time of VDC\nR8 from 470R to 1k to reduce current consumption blue voltage/therm/master LED (sufficient for EL357NC)\nFootprints same, still compatible with PCB 20210708 V1.0
+Text Notes 8200 7650 0    50   ~ 0
+2021-08-26      V1.1
 $EndSCHEMATC
